Commit message: Clarify EEF camera mounting frame name to prevent tf collisions
* update launch files
* update sim visualization window to show previous commits work

File: maze_support/urdf/eef_macro.xacro (robot description, xacro)
@@ -27,10 +27,10 @@
         <child link="${prefix}pointer_tcp"/>
     </joint>
-    <!-- Camera TCP defined as the tip of the expo marker -->
-    <link name="${prefix}camera_mnt"/>
-    <joint name="${prefix}eef_base_link-camera_mnt" type="fixed">
+    <!-- Camera Mount Point defined as the center of the mounting face -->
+    <link name="${prefix}eef_camera_mnt"/>
+    <joint name="${prefix}eef_base_link-eef_camera_mnt" type="fixed">
         <origin xyz="0.08300 0.01250 -0.02915" rpy="${radians(90)} ${radians(90)} 0"/>
         <parent link="${prefix}eef_base_link"/>
-        <child link="${prefix}camera_mnt"/>
+        <child link="${prefix}eef_camera_mnt"/>
     </joint>
 </xacro:macro>

File: maze_support/urdf/wc3.xacro (robot description, xacro)
@@ -15,5 +15,5 @@
     <xacro:arg name="use_nominal_extrinsics" default="false" />
     <xacro:include filename="$(find realsense2_description)/urdf/_d435i.urdf.xacro"/>
-    <xacro:sensor_d435i parent="camera_mnt" use_nominal_extrinsics="$(arg use_nominal_extrinsics)">
+    <xacro:sensor_d435i parent="eef_camera_mnt" use_nominal_extrinsics="$(arg use_nominal_extrinsics)">
         <origin xyz="0 0 0" rpy="0 0 0"/>
     </xacro:sensor_d435i>
